Commit message: Finished URDF model

File: src/robot_description/urdf/robot.urdf.xacro (robot description, xacro)
@@ -36,3 +36,77 @@
         <limit lower="-${PI/2}" upper="${PI/2}" effort="${EFFORT}" velocity="${VELOCITY}"/>
     </joint>
+    <link name="forward_drive_arm">
+        <visual>
+            <origin rpy="0 -${PI/2} ${PI/2}" xyz="0.19 0.06 -0.08"/>
+            <geometry>
+                <mesh filename="${FILE_PATH}/forward_drive_arm.STL" scale="0.01 0.01 0.01"/>
+            </geometry>
+        </visual>
+    </link>
+    <joint name="joint_2" type="revolute">
+        <parent link="base_plate"/>
+        <child link="forward_drive_arm"/>
+        <axis xyz="1 0 0"/>
+        <origin xyz="-0.02 0 0.35" rpy="0 0 0"/>
+        <limit lower="-${PI/2}" upper="${PI/2}" effort="${EFFORT}" velocity="${VELOCITY}"/>
+    </joint>
+    <link name="horizontal_arm">
+        <visual>
+            <origin rpy="${PI/2} 0 ${PI/2}" xyz="-0.03 -0.4 -0.06"/>
+            <geometry>
+                <mesh filename="${FILE_PATH}/horizontal_arm.STL" scale="0.01 0.01 0.01"/>
+            </geometry>
+        </visual>
+    </link>
+    <joint name="joint_3" type="revolute">
+        <parent link="forward_drive_arm"/>
+        <child link="horizontal_arm"/>
+        <axis xyz="1 0 0"/>
+        <origin rpy="0 0 0" xyz="0 0 0.8"/>
+        <limit lower="-${PI/2}" upper="${PI/2}" effort="${EFFORT}" velocity="${VELOCITY}"/>
+    </joint>
+    <link name="claw_support">
+        <visual>
+            <origin rpy="0 0 ${PI/2}" xyz="0 -0.05 -0.15"/>
+            <geometry>
+                <mesh filename="${FILE_PATH}/claw_support.STL" scale="0.01 0.01 0.01"/>
+            </geometry>
+        </visual>
+    </link>
+    <joint name="horizontal_arm_to_claw_support" type="fixed">
+        <parent link="horizontal_arm"/>
+        <child link="claw_support"/>
+        <origin rpy="0 0 0" xyz="0 0.82 0"/>
+    </joint>
+    <link name="gripper_right">
+        <visual>
+            <origin rpy="0 0 -${PI/2}" xyz="-0.1 0.5 -0.1"/>
+            <geometry>
+                <mesh filename="${FILE_PATH}/right_finger.STL" scale="0.01 0.01 0.01"/>
+            </geometry>
+        </visual>
+    </link>
+    <link name="gripper_left">
+        <visual>
+            <origin rpy="0 0 -${PI/2}" xyz="-0.04 0.5 -0.1"/>
+            <geometry>
+                <mesh filename="${FILE_PATH}/left_finger.STL" scale="0.01 0.01 0.01"/>
+            </geometry>
+        </visual>
+    </link>
+    <joint name="joint_4" type="revolute">
+        <parent link="claw_support"/>
+        <child link="gripper_right"/>
+        <axis xyz="0 0 1"/>
+        <origin rpy="0 0 0" xyz="-0.04 0.13 -0.1"/>
+        <limit lower="-${PI/2}" upper="0.0" effort="${EFFORT}" velocity="${VELOCITY}"/>
+    </joint>
+    <joint name="joint_5" type="revolute">
+        <parent link="claw_support"/>
+        <child link="gripper_left"/>
+        <axis xyz="0 0 1"/>
+        <origin rpy="0 0 0" xyz="-0.22 0.13 -0.1"/>
+        <mimic joint="joint_4" multiplier="-1"/>
+        <limit lower="0.0" upper="${PI/2}" effort="${EFFORT}" velocity="${VELOCITY}"/>
+    </joint>
 </robot>

Commit message: collision tag content updated

File: src/robot_description/urdf/robot.urdf.xacro (robot description, xacro)
@@ -14,4 +14,10 @@
             </geometry>
         </visual>
+        <collision>
+            <origin rpy="0 0 0" xyz="-0.5 -0.5 0"/>
+            <geometry>
+                <mesh filename="${FILE_PATH}/basement.STL" scale="0.01 0.01 0.01"/>
+            </geometry>
+        </collision>
     </link>
     <link name="base_plate">
@@ -22,4 +28,10 @@
             </geometry>
         </visual>
+        <collision>
+            <origin rpy="0 0 0" xyz="-0.39 -0.39 -0.56"/>
+            <geometry>
+                <mesh filename="${FILE_PATH}/base_plate.STL" scale="0.01 0.01 0.01"/>
+            </geometry>
+        </collision>
     </link>
     <!-- Joints -->
@@ -43,4 +55,10 @@
             </geometry>
         </visual>
+        <collision>
+            <origin rpy="0 -${PI/2} ${PI/2}" xyz="0.19 0.06 -0.08"/>
+            <geometry>
+                <mesh filename="${FILE_PATH}/forward_drive_arm.STL" scale="0.01 0.01 0.01"/>
+            </geometry>
+        </collision>
     </link>
     <joint name="joint_2" type="revolute">
@@ -58,4 +76,10 @@
             </geometry>
         </visual>
+        <collision>
+            <origin rpy="${PI/2} 0 ${PI/2}" xyz="-0.03 -0.4 -0.06"/>
+            <geometry>
+                <mesh filename="${FILE_PATH}/horizontal_arm.STL" scale="0.01 0.01 0.01"/>
+            </geometry>
+        </collision>
     </link>
     <joint name="joint_3" type="revolute">
@@ -73,4 +97,10 @@
             </geometry>
         </visual>
+        <collision>
+            <origin rpy="0 0 ${PI/2}" xyz="0 -0.05 -0.15"/>
+            <geometry>
+                <mesh filename="${FILE_PATH}/claw_support.STL" scale="0.01 0.01 0.01"/>
+            </geometry>
+        </collision>
     </link>
     <joint name="horizontal_arm_to_claw_support" type="fixed">
@@ -86,4 +116,10 @@
             </geometry>
         </visual>
+        <collision>
+             <origin rpy="0 0 -${PI/2}" xyz="-0.1 0.5 -0.1"/>
+            <geometry>
+                <mesh filename="${FILE_PATH}/right_finger.STL" scale="0.01 0.01 0.01"/>
+            </geometry>
+        </collision>
     </link>
     <link name="gripper_left">
@@ -94,4 +130,10 @@
             </geometry>
         </visual>
+        <collision>
+            <origin rpy="0 0 -${PI/2}" xyz="-0.04 0.5 -0.1"/>
+            <geometry>
+                <mesh filename="${FILE_PATH}/left_finger.STL" scale="0.01 0.01 0.01"/>
+            </geometry>
+        </collision>
     </link>
     <joint name="joint_4" type="revolute">

Commit message: inertia values assigned to links

File: src/robot_description/urdf/robot.urdf.xacro (robot description, xacro)
@@ -5,7 +5,16 @@
     <xacro:property name="EFFORT" value="30.0"/>
     <xacro:property name="FILE_PATH" value="file://$(find robot_description)/meshes"/>
+    <xacro:macro name="default_inertial" params="mass">
+        <inertial>
+            <mass value="${mass}"/>
+            <innertia ixx="1.0" ixy="0.0" ixz="0.0"
+                      iyy="1.0" iyz="0.0"
+                      izz="1.0"/>
+        </inertial>
+    </xacro:macro>
     <!-- Links -->
     <link name="world"/>
     <link name="base_link">
+        <xacro:default_inertial mass="1"/>
         <visual>
             <origin rpy="0 0 0" xyz="-0.5 -0.5 0"/>
@@ -22,4 +31,5 @@
     </link>
     <link name="base_plate">
+    <xacro:default_inertial mass="0.1"/>
         <visual>
             <origin rpy="0 0 0" xyz="-0.39 -0.39 -0.56"/>
@@ -49,4 +59,5 @@
     </joint>
     <link name="forward_drive_arm">
+    <xacro:default_inertial mass="0.1"/>
         <visual>
             <origin rpy="0 -${PI/2} ${PI/2}" xyz="0.19 0.06 -0.08"/>
@@ -70,4 +81,5 @@
     </joint>
     <link name="horizontal_arm">
+        <xacro:default_inertial mass="0.1"/>
         <visual>
             <origin rpy="${PI/2} 0 ${PI/2}" xyz="-0.03 -0.4 -0.06"/>
@@ -91,4 +103,5 @@
     </joint>
     <link name="claw_support">
+        <xacro:default_inertial mass="0.05"/>
         <visual>
             <origin rpy="0 0 ${PI/2}" xyz="0 -0.05 -0.15"/>
@@ -110,4 +123,5 @@
     </joint>
     <link name="gripper_right">
+        <xacro:default_inertial mass="0.01"/>
         <visual>
             <origin rpy="0 0 -${PI/2}" xyz="-0.1 0.5 -0.1"/>
@@ -124,4 +138,5 @@
     </link>
     <link name="gripper_left">
+        <xacro:default_inertial mass="0.01"/>
         <visual>
             <origin rpy="0 0 -${PI/2}" xyz="-0.04 0.5 -0.1"/>

Commit message: minor issues corrected

File: src/robot_description/urdf/robot.urdf.xacro (robot description, xacro)
@@ -8,5 +8,5 @@
         <inertial>
             <mass value="${mass}"/>
-            <innertia ixx="1.0" ixy="0.0" ixz="0.0"
+            <inertia ixx="1.0" ixy="0.0" ixz="0.0"
                       iyy="1.0" iyz="0.0"
                       izz="1.0"/>

Commit message: Refactored urdf file

File: src/robot_description/urdf/robot.urdf.xacro (robot description, xacro)
@@ -45,39 +45,19 @@
         </collision>
     </link>
-    <!-- Joints -->
-    <joint name="virtual_joint" type="fixed">
-        <parent link="world"/>
-        <child link="base_link"/>
-        <origin xyz="0 0 0" rpy="0 0 0"/>
-    </joint>
-    <joint name="joint_1" type="revolute">
-        <parent link="base_link"/>
-        <child link="base_plate"/>
-        <axis xyz="0 0 1"/>
-        <origin xyz="0 0 0.307" rpy="0 0 0"/>
-        <limit lower="-${PI/2}" upper="${PI/2}" effort="${EFFORT}" velocity="${VELOCITY}"/>
-    </joint>
     <link name="forward_drive_arm">
-    <xacro:default_inertial mass="0.1"/>
-        <visual>
-            <origin rpy="0 -${PI/2} ${PI/2}" xyz="0.19 0.06 -0.08"/>
-            <geometry>
-                <mesh filename="${FILE_PATH}/forward_drive_arm.STL" scale="0.01 0.01 0.01"/>
-            </geometry>
-        </visual>
-        <collision>
-            <origin rpy="0 -${PI/2} ${PI/2}" xyz="0.19 0.06 -0.08"/>
-            <geometry>
-                <mesh filename="${FILE_PATH}/forward_drive_arm.STL" scale="0.01 0.01 0.01"/>
-            </geometry>
-        </collision>
+        <xacro:default_inertial mass="0.1"/>
+            <visual>
+                <origin rpy="0 -${PI/2} ${PI/2}" xyz="0.19 0.06 -0.08"/>
+                <geometry>
+                    <mesh filename="${FILE_PATH}/forward_drive_arm.STL" scale="0.01 0.01 0.01"/>
+                </geometry>
+            </visual>
+            <collision>
+                <origin rpy="0 -${PI/2} ${PI/2}" xyz="0.19 0.06 -0.08"/>
+                <geometry>
+                    <mesh filename="${FILE_PATH}/forward_drive_arm.STL" scale="0.01 0.01 0.01"/>
+                </geometry>
+            </collision>
     </link>
-    <joint name="joint_2" type="revolute">
-        <parent link="base_plate"/>
-        <child link="forward_drive_arm"/>
-        <axis xyz="1 0 0"/>
-        <origin xyz="-0.02 0 0.35" rpy="0 0 0"/>
-        <limit lower="-${PI/2}" upper="${PI/2}" effort="${EFFORT}" velocity="${VELOCITY}"/>
-    </joint>
     <link name="horizontal_arm">
         <xacro:default_inertial mass="0.1"/>
@@ -95,11 +75,4 @@
         </collision>
     </link>
-    <joint name="joint_3" type="revolute">
-        <parent link="forward_drive_arm"/>
-        <child link="horizontal_arm"/>
-        <axis xyz="1 0 0"/>
-        <origin rpy="0 0 0" xyz="0 0 0.8"/>
-        <limit lower="-${PI/2}" upper="${PI/2}" effort="${EFFORT}" velocity="${VELOCITY}"/>
-    </joint>
     <link name="claw_support">
         <xacro:default_inertial mass="0.05"/>
@@ -117,9 +90,4 @@
         </collision>
     </link>
-    <joint name="horizontal_arm_to_claw_support" type="fixed">
-        <parent link="horizontal_arm"/>
-        <child link="claw_support"/>
-        <origin rpy="0 0 0" xyz="0 0.82 0"/>
-    </joint>
     <link name="gripper_right">
         <xacro:default_inertial mass="0.01"/>
@@ -152,4 +120,36 @@
         </collision>
     </link>
+    <!-- Joints -->
+    <joint name="virtual_joint" type="fixed">
+        <parent link="world"/>
+        <child link="base_link"/>
+        <origin xyz="0 0 0" rpy="0 0 0"/>
+    </joint>
+    <joint name="joint_1" type="revolute">
+        <parent link="base_link"/>
+        <child link="base_plate"/>
+        <axis xyz="0 0 1"/>
+        <origin xyz="0 0 0.307" rpy="0 0 0"/>
+        <limit lower="-${PI/2}" upper="${PI/2}" effort="${EFFORT}" velocity="${VELOCITY}"/>
+    </joint>
+    <joint name="joint_2" type="revolute">
+        <parent link="base_plate"/>
+        <child link="forward_drive_arm"/>
+        <axis xyz="1 0 0"/>
+        <origin xyz="-0.02 0 0.35" rpy="0 0 0"/>
+        <limit lower="-${PI/2}" upper="${PI/2}" effort="${EFFORT}" velocity="${VELOCITY}"/>
+    </joint>
+    <joint name="joint_3" type="revolute">
+        <parent link="forward_drive_arm"/>
+        <child link="horizontal_arm"/>
+        <axis xyz="1 0 0"/>
+        <origin rpy="0 0 0" xyz="0 0 0.8"/>
+        <limit lower="-${PI/2}" upper="${PI/2}" effort="${EFFORT}" velocity="${VELOCITY}"/>
+    </joint>
+    <joint name="horizontal_arm_to_claw_support" type="fixed">
+        <parent link="horizontal_arm"/>
+        <child link="claw_support"/>
+        <origin rpy="0 0 0" xyz="0 0.82 0"/>
+    </joint>
     <joint name="joint_4" type="revolute">
         <parent link="claw_support"/>

Commit message: oriented rpi camera

File: src/robot_description/urdf/robot.urdf.xacro (robot description, xacro)
@@ -120,4 +120,19 @@
         </collision>
     </link>
+    <link name="rgb_camera">
+        <xacro:default_inertia mass="0.001"/>
+        <visual>
+            <origin rpy="-${PI/2} 0 -${PI/2}" xyz="-0.1 0.13 0.13"/>
+            <geometry>
+                <mesh filename="${FILE_PATH}/pi_camera.STL" scale="0.01 0.01 0.01"/>
+            </geometry>
+        </visual>
+        <collision>
+            <origin rpy="-${PI/2} 0 -${PI/2}" xyz="-0.1 0.13 0.13"/>
+            <geometry>
+                <mesh filename="${FILE_PATH}/pi_camera.STL" scale="0.01 0.01 0.01"/>
+            </geometry>
+        </collision>
+    </link>
     <!-- Joints -->
     <joint name="virtual_joint" type="fixed">
@@ -125,4 +140,9 @@
         <child link="base_link"/>
         <origin xyz="0 0 0" rpy="0 0 0"/>
+    </joint>
+    <joint name="rgb_camera_joint" type="fixed">
+        <parent link="base_link"/>
+        <child link="rgb_camera"/>
+        <origin xyz="0 0.45 0.2" rpy="0 -${PI/6} 1.57"/>
     </joint>
     <joint name="joint_1" type="revolute">
